Commit message: blacklisted pts, params, turtlebot

File: mae_simulator/urdf/mav_generic_odometry_and_lidar.xacro (robot description, xacro)
@@ -58,5 +58,6 @@
       noise="0.008"
       min_angle="-${M_PI}"
-      max_angle="${M_PI}">
+      max_angle="${M_PI}"
+      namespace="${namespace}">
       <origin xyz="0.0 0 -0.12" rpy="0.0 0.0 0.0" />
     </xacro:VLP-16>

File: velodyne_simulator/velodyne_description/urdf/VLP-16.urdf.xacro (robot description, xacro)
@@ -2,5 +2,5 @@
 <robot xmlns:xacro="http://www.ros.org/wiki/xacro" name="VLP-16">
   <xacro:property name="M_PI" value="3.1415926535897931" />
-  <xacro:macro name="VLP-16" params="*origin parent:=base_link name:=velodyne topic:=/velodyne_points hz:=10 lasers:=16 samples:=1875 collision_range:=0.3 min_range:=0.9 max_range:=130.0 noise:=0.008 min_angle:=-${M_PI} max_angle:=${M_PI} gpu:=false">
+  <xacro:macro name="VLP-16" params="*origin parent:=base_link name:=velodyne topic:=/velodyne_points hz:=10 lasers:=16 samples:=1875 collision_range:=0.3 min_range:=0.9 max_range:=130.0 noise:=0.008 min_angle:=-${M_PI} max_angle:=${M_PI} gpu:=false namespace:=test">
     <joint name="${namespace}/${name}_base_mount_joint" type="fixed">
       <xacro:insert_block name="origin" />
